Commit message: Description: Correction of plain urdf, added launches and rviz config

File: diff_robot_dan_description/urdf/diff_robot_dan.urdf (robot description, URDF)
Before this commit: robot diff_robot_dan, 39 links, 38 joints
Joints:
- joint central_wheel_to_shaft: axis -1 0 0 -> 0 0 0; type continuous -> fixed
- joint motor_right_to_support: origin xyz=0 -0.01155 0.02025 rpy=1.5708 1.5708 0 -> xyz=0 -0.01155 0.02025 rpy=1.5708 1.5708 -3.1416
- joint roll_support_to_wheel_support: axis 0 0 0 -> 0 1 0; type fixed -> continuous
- joint shaft_to_roll_support: axis 0 0 0 -> 0 0 1; origin xyz=-0.016111 0.018272 4.708E-05 rpy=0 0 -0.77638 -> xyz=-0.016111 0.018272 4.708E-05 rpy=0 0 0
