Commit message: Description: Adding launch.py for manual visualization

File: diff_robot_dan_description/urdf/diff_robot_dan.urdf.xacro (robot description, xacro)
@@ -1268,4 +1268,16 @@
       xyz="0 1 0" />
   </joint>
+  <joint
+    name="shaft_to_roll_support"
+    type="continuous">
+    <origin
+      xyz="-0.016111 0.018272 4.708E-05"
+      rpy="0 0 0" />
+    <parent
+      link="roll_support" />
+    <child
+      link="central_shaft" />
+    <axis
+      xyz="0 0 1" />
   <link
     name="central_shaft">
@@ -1308,16 +1320,4 @@
     </collision>
   </link>
-  <joint
-    name="shaft_to_roll_support"
-    type="continuous">
-    <origin
-      xyz="-0.016111 0.018272 4.708E-05"
-      rpy="0 0 0" />
-    <parent
-      link="roll_support" />
-    <child
-      link="central_shaft" />
-    <axis
-      xyz="0 0 1" />
   </joint>
   <link
