Commit message: Description and Gazebo: Adding controller, and starting to move the robot (move still needs improvements)

File: diff_robot_dan_description/urdf/diff_robot_dan.xacro (robot description, xacro)
@@ -3,3 +3,4 @@
     <xacro:include filename="$(find diff_robot_dan_description)/urdf/diff_robot_dan_core.urdf.xacro"/>
     <xacro:include filename="$(find diff_robot_dan_description)/urdf/diff_robot_dan_gazebo.xacro"/>
+    <xacro:include filename="$(find diff_robot_dan_description)/urdf/diff_robot_dan_controllers.xacro"/>
 </robot>

File: diff_robot_dan_description/urdf/diff_robot_dan_gazebo.xacro (robot description, xacro)
@@ -1,24 +1,51 @@
 <?xml version="1.0"?>
 <robot xmlns:xacro="http://www.ros.org/wiki/xacro"  name="diff_robot_dan_gazebo">
+    <!-- ____________________ Macro definitions ______________________-->
+    <xacro:macro name="wheel_material_def" params="side">
+        <gazebo reference="motor_support_${side}">
+        <material>Gazebo/Black</material>
+        </gazebo>
+        <gazebo reference="motor_${side}">
+            <material>Gazebo/Grey</material>
+        </gazebo>
+        <gazebo reference="shaft_${side}">
+            <material>Gazebo/Grey</material>
+        </gazebo>
+        <gazebo reference="coupling_${side}">
+            <material>Gazebo/Gold</material>
+        </gazebo>
+        <gazebo reference="ring_${side}">
+            <material>Gazebo/Blue</material>
+        </gazebo>
+        <gazebo reference="neumatic_${side}">
+            <material>Gazebo/DarkGrey</material>
+        </gazebo>
+    </xacro:macro>
+    <xacro:macro name="small_hex_material" params="num">
+        <gazebo reference="hex_support_s${num}">
+            <material>Gazebo/Gold</material>
+        </gazebo>
+    </xacro:macro>
+    <xacro:macro name="medium_hex_material" params="num">
+        <gazebo reference="hex_support_m${num}">
+            <material>Gazebo/Gold</material>
+        </gazebo>
+    </xacro:macro>
+    <!-- ____________________ Macro implementations ______________________-->
+    <xacro:wheel_material_def side="left"/>
+    <xacro:wheel_material_def side="right"/>
+    <xacro:small_hex_material num="1"/>
+    <xacro:small_hex_material num="2"/>
+    <xacro:small_hex_material num="3"/>
+    <xacro:small_hex_material num="4"/>
+    <xacro:medium_hex_material num="1"/>
+    <xacro:medium_hex_material num="2"/>
+    <xacro:medium_hex_material num="3"/>
+    <xacro:medium_hex_material num="4"/>
+    <xacro:medium_hex_material num="5"/>
+    <xacro:medium_hex_material num="6"/>
+    <!-- ____________________ Other definitions __________________________-->
     <gazebo reference="base_platform">
-        <material>Gazebo/DarkGrey</material>
-    </gazebo>
-    <gazebo reference="motor_support_left">
-        <material>Gazebo/Black</material>
-    </gazebo>
-    <gazebo reference="motor_left">
         <material>Gazebo/Grey</material>
-    </gazebo>
-    <gazebo reference="shaft_left">
-        <material>Gazebo/Grey</material>
-    </gazebo>
-    <gazebo reference="coupling_left">
-        <material>Gazebo/Gold</material>
-    </gazebo>
-    <gazebo reference="ring_left">
-        <material>Gazebo/Blue</material>
-    </gazebo>
-    <gazebo reference="neumatic_left">
-        <material>Gazebo/Black</material>
     </gazebo>
     <gazebo reference="battery_holder">
@@ -37,16 +64,4 @@
         <material>Gazebo/Red</material>
     </gazebo>
-    <gazebo reference="hex_support_s1">
-        <material>Gazebo/Gold</material>
-    </gazebo>
-    <gazebo reference="hex_support_s2">
-        <material>Gazebo/Gold</material>
-    </gazebo>
-    <gazebo reference="hex_support_s3">
-        <material>Gazebo/Gold</material>
-    </gazebo>
-    <gazebo reference="hex_support_s4">
-        <material>Gazebo/Gold</material>
-    </gazebo>
     <gazebo reference="center_wheel_support">
         <material>Gazebo/DarkGrey</material>
@@ -58,5 +73,5 @@
         <material>Gazebo/DarkGrey</material>
     </gazebo>
-    <gazebo reference="center_wheel">
+    <gazebo reference="central_wheel">
         <material>Gazebo/Black</material>
     </gazebo>
@@ -82,21 +97,3 @@
         <material>Gazebo/DarkGrey</material>
     </gazebo>
-    <gazebo reference="hex_support_m1">
-        <material>Gazebo/Gold</material>
-    </gazebo>
-    <gazebo reference="hex_support_m2">
-        <material>Gazebo/Gold</material>
-    </gazebo>
-    <gazebo reference="hex_support_m3">
-        <material>Gazebo/Gold</material>
-    </gazebo>
-    <gazebo reference="hex_support_m4">
-        <material>Gazebo/Gold</material>
-    </gazebo>
-    <gazebo reference="hex_support_m5">
-        <material>Gazebo/Gold</material>
-    </gazebo>
-    <gazebo reference="hex_support_m6">
-        <material>Gazebo/Gold</material>
-    </gazebo>
 </robot>

Commit message: Description and Gazebo: Correcting collision and spawn pose

File: diff_robot_dan_description/urdf/diff_robot_dan.xacro (robot description, xacro)
@@ -1,8 +1,13 @@
 <?xml version="1.0"?>
 <robot xmlns:xacro="http://www.ros.org/wiki/xacro"  name="diff_robot_dan">
+    <xacro:arg name="use_ros2_control" default="true"/>
     <xacro:include filename="$(find diff_robot_dan_description)/urdf/diff_robot_dan_core.urdf.xacro"/>
+    <xacro:if value="$(arg use_ros2_control)">
+        <xacro:include filename="$(find diff_robot_dan_description)/urdf/diff_robot_dan_ros2_control.xacro"/>
+    </xacro:if>
+    <xacro:unless value="$(arg use_ros2_control)">
+        <xacro:include filename="$(find diff_robot_dan_description)/urdf/diff_robot_dan_controllers.xacro"/>
+    </xacro:unless>
     <xacro:include filename="$(find diff_robot_dan_description)/urdf/diff_robot_dan_gazebo.xacro"/>
-    <xacro:include filename="$(find diff_robot_dan_description)/urdf/diff_robot_dan_ros2_control.xacro"/>
-    <!--xacro:include filename="$(find diff_robot_dan_description)/urdf/diff_robot_dan_controllers.xacro"/-->
     <xacro:include filename="$(find diff_robot_dan_description)/urdf/diff_robot_dan_sensors.xacro"/>
 </robot>

File: diff_robot_dan_description/urdf/diff_robot_dan_core.urdf.xacro (robot description, xacro)
@@ -2,4 +2,5 @@
 <robot xmlns:xacro="http://www.ros.org/wiki/xacro">
   <xacro:include filename="$(find diff_robot_dan_description)/urdf/materials_and_colors.xacro"/>
+  <xacro:property name="caster_type" value="continuous" />
   <link name="base_link"/>
   <link
@@ -1174,5 +1175,5 @@
   <joint
     name="roll_support_to_wheel_support"
-    type="continuous">
+    type="${caster_type}">
     <origin
       xyz="0 0.004693 0"
@@ -1223,5 +1224,5 @@
   <joint
     name="shaft_to_roll_support"
-    type="continuous">
+    type="${caster_type}">
     <origin
       xyz="-0.016111 0.018272 4.708E-05"
@@ -1606,5 +1607,5 @@
       <origin
         xyz="0 0 0"
-        rpy="0 0 0" />
+        rpy="0 0 1.5707" />
       <geometry>
         <mesh

File: diff_robot_dan_description/urdf/diff_robot_dan_sensors.xacro (robot description, xacro)
@@ -2,19 +2,9 @@
 <robot xmlns:xacro="http://www.ros.org/wiki/xacro">
     <link name="laser_frame">
-        <visual>
-            <geometry>
-                <cylinder length="0.005" radius="0.005"/>
-            </geometry>
-        </visual>
-        <collision>
-            <geometry>
-                <cylinder length="0.01" radius="0.02"/>
-            </geometry>
-        </collision>
     </link>
     <joint name="laser_joint" type="fixed">
         <parent link="lidar_base"/>
         <child link="laser_frame"/>
-        <origin xyz="0 0 0.035" rpy="0 0 0"/>
+        <origin xyz="0 0 0.0445" rpy="0 0 1.57"/>
     </joint>
     <gazebo reference="laser_frame">
@@ -47,5 +37,7 @@
             <plugin name="scan" filename="libgazebo_ros_ray_sensor.so">
                 <ros>
-                    <argument>~/out:=/scan</argument>
+                    <argument>--ros-args</argument>
+                    <argument>-r</argument>
+                    <argument>~/out:=scan</argument>
                 </ros>
                 <output_type>sensor_msgs/LaserScan</output_type>
