Commit message: Description: Correcting axis of transform for making rotation only on z axis on shafts

File: diff_robot_dan_description/urdf/diff_robot_dan_controllers.xacro (robot description, xacro)
@@ -2,23 +2,23 @@
 <robot xmlns:xacro="http://www.ros.org/wiki/xacro">
     <gazebo reference="central_wheel">
-        <mu1 value="0.001"/>
-        <mu2 value="0.001"/>
+        <mu1 value="0.0"/>
+        <mu2 value="0.0"/>
     </gazebo>
     <gazebo reference="neumatic_right">
         <mu1 value="0.1"/>
         <mu2 value="0.1"/>
-        <kp>500000.0</kp>
-        <kd>10.0</kd>
+        <kp>1.0</kp>
+        <kd>0.0</kd>
         <minDepth>0.001</minDepth>
-        <maxVel>0.1</maxVel>
+        <maxVel>0.2</maxVel>
     </gazebo>
-    <gazebo reference="neumatic_left">
+    <!gazebo reference="neumatic_left">
         <mu1 value="0.1"/>
         <mu2 value="0.1"/>
-        <kp>500000.0</kp>
-        <kd>10.0</kd>
+        <kp>1.0</kp>
+        <kd>0.0</kd>
         <minDepth>0.001</minDepth>
-        <maxVel>0.1</maxVel>
-    </gazebo>
+        <maxVel>0.2</maxVel>
+    </!gazebo>
     <gazebo>
         <plugin name="diff_drive" filename="libgazebo_ros_diff_drive.so">

File: diff_robot_dan_description/urdf/diff_robot_dan_core.urdf.xacro (robot description, xacro)
@@ -53,4 +53,13 @@
       xyz="0 0 0" />
   </joint>
+  <link name="base_footprint"/>
+  <joint name="to_footprint" type="fixed">
+    <parent
+      link="base_platform"/>
+    <child
+      link="base_footprint"/>
+    <axis
+      xyz="0.0 0.0 0.0"/>
+  </joint>
   <link
     name="motor_support_left">
@@ -222,5 +231,5 @@
       <origin
         xyz="0 0 0"
-        rpy="0 0 0" />
+        rpy="1.5708 0 0" />
       <geometry>
         <mesh
@@ -232,5 +241,5 @@
       <origin
         xyz="0 0 0"
-        rpy="0 0 0" />
+        rpy="1.5708 0 0" />
       <geometry>
         <mesh
@@ -244,5 +253,5 @@
     <origin
       xyz="0 0 0.0046"
-      rpy="1.5708 0 1.7908" />
+      rpy="0 0 1.7908" />
     <parent
       link="shaft_left" />
@@ -271,5 +280,5 @@
       <origin
         xyz="0 0 0"
-        rpy="0 0 0" />
+        rpy="-1.5708 0 0" />
       <geometry>
         <mesh
@@ -281,5 +290,5 @@
       <origin
         xyz="0 0 0"
-        rpy="0 0 0" />
+        rpy="-1.5708 0 0" />
       <geometry>
         <mesh
@@ -292,6 +301,6 @@
     type="fixed">
     <origin
-      xyz="0 0.021355 0"
-      rpy="3.1416 0 0" />
+      xyz="0 0 0.021355"
+      rpy="0 0 0" />
     <parent
       link="coupling_left" />
@@ -320,5 +329,5 @@
       <origin
         xyz="0 0 0"
-        rpy="0 0 0" />
+        rpy="1.5708 0 0" />
       <geometry>
         <mesh
@@ -330,7 +339,9 @@
       <origin
         xyz="0 0 0"
-        rpy="0 0 0" />
-      <geometry>
-        <sphere radius="0.03394"/>
+        rpy="1.5708 0 0" />
+      <geometry>
+        <!--sphere radius="0.03394"/-->
+        <mesh
+          filename="package://diff_robot_dan_description/meshes/neumatic_left.STL" />
       </geometry>
     </collision>
@@ -340,6 +351,6 @@
     type="fixed">
     <origin
-      xyz="-8.7612E-05 0.00055 4.2289E-05"
-      rpy="-3.1416 -0.4497 3.1416" />
+      xyz="0 0.00055 0"
+      rpy="0 0 0" />
     <parent
       link="ring_left" />
@@ -518,5 +529,5 @@
       <origin
         xyz="0 0 0"
-        rpy="0 0 0" />
+        rpy="1.5708 0 0" />
       <geometry>
         <mesh
@@ -528,5 +539,5 @@
       <origin
         xyz="0 0 0"
-        rpy="0 0 0" />
+        rpy="1.5708 0 0" />
       <geometry>
         <mesh
@@ -540,5 +551,5 @@
     <origin
       xyz="0 0 0.0046"
-      rpy="1.5708 0 -1.7908" />
+      rpy="0 0 -1.7908" />
     <parent
       link="shaft_right" />
@@ -567,5 +578,5 @@
       <origin
         xyz="0 0 0"
-        rpy="0 0 0" />
+        rpy="-1.5708 0 0" />
       <geometry>
         <mesh
@@ -577,5 +588,5 @@
       <origin
         xyz="0 0 0"
-        rpy="0 0 0" />
+        rpy="-1.5708 0 0" />
       <geometry>
         <mesh
@@ -588,6 +599,6 @@
     type="fixed">
     <origin
-      xyz="0 0.021355 0"
-      rpy="3.1416 0 0" />
+      xyz="0 0 0.021355"
+      rpy="0 0 0" />
     <parent
       link="coupling_right" />
@@ -616,5 +627,5 @@
       <origin
         xyz="0 0 0"
-        rpy="0 0 0" />
+        rpy="1.5708 0 0" />
       <geometry>
         <mesh
@@ -626,7 +637,9 @@
       <origin
         xyz="0 0 0"
-        rpy="0 0 0" />
-      <geometry>
-        <sphere radius="0.03394"/>
+        rpy="1.5708 0 0" />
+      <geometry>
+        <!--sphere radius="0.03394"/-->
+        <mesh
+          filename="package://diff_robot_dan_description/meshes/neumatic_right.STL" />
       </geometry>
     </collision>
@@ -637,5 +650,5 @@
     <origin
       xyz="0 0.00055 0"
-      rpy="0 -0.4497 0" />
+      rpy="0 0 0" />
     <parent
       link="ring_right" />
@@ -1264,5 +1277,7 @@
         rpy="0 0 0" />
       <geometry>
-        <sphere radius="0.0127"/>
+        <!--sphere radius="0.0127"/-->
+        <mesh
+          filename="package://diff_robot_dan_description/meshes/central_wheel.STL" />
       </geometry>
     </collision>

Commit message: Description and Gazebo: Modifying friction and collision of wheels, odomettry improved angular but linear still fails, movement improved

File: diff_robot_dan_description/urdf/diff_robot_dan_controllers.xacro (robot description, xacro)
@@ -1,24 +1,4 @@
 <?xml version="1.0"?>
 <robot xmlns:xacro="http://www.ros.org/wiki/xacro">
-    <gazebo reference="central_wheel">
-        <mu1 value="0.0"/>
-        <mu2 value="0.0"/>
-    </gazebo>
-    <gazebo reference="neumatic_right">
-        <mu1 value="0.1"/>
-        <mu2 value="0.1"/>
-        <kp>1.0</kp>
-        <kd>0.0</kd>
-        <minDepth>0.001</minDepth>
-        <maxVel>0.2</maxVel>
-    </gazebo>
-    <!gazebo reference="neumatic_left">
-        <mu1 value="0.1"/>
-        <mu2 value="0.1"/>
-        <kp>1.0</kp>
-        <kd>0.0</kd>
-        <minDepth>0.001</minDepth>
-        <maxVel>0.2</maxVel>
-    </!gazebo>
     <gazebo>
         <plugin name="diff_drive" filename="libgazebo_ros_diff_drive.so">

File: diff_robot_dan_description/urdf/diff_robot_dan_core.urdf.xacro (robot description, xacro)
@@ -341,7 +341,7 @@
         rpy="1.5708 0 0" />
       <geometry>
-        <!--sphere radius="0.03394"/-->
-        <mesh
-          filename="package://diff_robot_dan_description/meshes/neumatic_left.STL" />
+        <sphere radius="0.03394"/>
+        <!--mesh
+          filename="package://diff_robot_dan_description/meshes/neumatic_left.STL" /-->
       </geometry>
     </collision>
@@ -639,7 +639,7 @@
         rpy="1.5708 0 0" />
       <geometry>
-        <!--sphere radius="0.03394"/-->
-        <mesh
-          filename="package://diff_robot_dan_description/meshes/neumatic_right.STL" />
+        <sphere radius="0.03394"/>
+        <!--mesh
+          filename="package://diff_robot_dan_description/meshes/neumatic_right.STL" /-->
       </geometry>
     </collision>
@@ -1277,7 +1277,7 @@
         rpy="0 0 0" />
       <geometry>
-        <!--sphere radius="0.0127"/-->
-        <mesh
-          filename="package://diff_robot_dan_description/meshes/central_wheel.STL" />
+        <sphere radius="0.0127"/>
+        <!--mesh
+          filename="package://diff_robot_dan_description/meshes/central_wheel.STL" /-->
       </geometry>
     </collision>

File: diff_robot_dan_description/urdf/diff_robot_dan_gazebo.xacro (robot description, xacro)
@@ -97,3 +97,23 @@
         <material>Gazebo/DarkGrey</material>
     </gazebo>
+    <gazebo reference="central_wheel">
+        <mu1 value="0.01"/>
+        <mu2 value="0.01"/>
+    </gazebo>
+    <gazebo reference="neumatic_right">
+        <mu1 value="0.1"/>
+        <mu2 value="0.1"/>
+        <kp>1.0</kp>
+        <kd>0.0</kd>
+        <minDepth>0.001</minDepth>
+        <maxVel>0.2</maxVel>
+    </gazebo>
+    <gazebo reference="neumatic_left">
+        <mu1 value="0.1"/>
+        <mu2 value="0.1"/>
+        <kp>1.0</kp>
+        <kd>0.0</kd>
+        <minDepth>0.001</minDepth>
+        <maxVel>0.2</maxVel>
+    </gazebo>
 </robot>
