Commit message: Description and Bringup: Correcting laser frame and adding slam params

File: diff_robot_dan_description/urdf/diff_robot_dan_sensors.xacro (robot description, xacro)
@@ -6,5 +6,7 @@
         <parent link="lidar_base"/>
         <child link="laser_frame"/>
-        <origin xyz="0 0 0.0445" rpy="0 0 1.57"/>
+        <origin
+            xyz="0 0 0.0445"
+            rpy="0 0 -1.57"/>
     </joint>
     <gazebo reference="laser_frame">
