Commit message: Description: Adding xacro file for colors and materials, improving core xacro and adding new Rviz config

File: diff_robot_dan_description/urdf/diff_robot_dan_core.urdf.xacro (robot description, xacro)
@@ -3,4 +3,5 @@
   name="diff_robot_dan_description_core"
   xmlns:xacro="http://www.ros.org/wiki/xacro">
+  <xacro:include filename="$(find diff_robot_dan_description)/urdf/materials_and_colors.xacro"/>
   <link name="base_link"/>
   <link
@@ -28,9 +29,5 @@
           filename="package://diff_robot_dan_description/meshes/base_platform.STL" />
       </geometry>
-      <material
-        name="">
-        <color
-          rgba="0.75294 0.75294 0.75294 1" />
-      </material>
+      <material name="grey_pla"/>
     </visual>
     <collision>
@@ -81,9 +78,5 @@
           filename="package://diff_robot_dan_description/meshes/motor_support_left.STL" />
       </geometry>
-      <material
-        name="">
-        <color
-          rgba="0.89804 0.91765 0.92941 1" />
-      </material>
+      <material name="black"/>
     </visual>
     <collision>
@@ -134,9 +127,5 @@
           filename="package://diff_robot_dan_description/meshes/motor_left.STL" />
       </geometry>
-      <material
-        name="">
-        <color
-          rgba="0.89804 0.91765 0.92941 1" />
-      </material>
+      <material name="silver_metal"/>
     </visual>
     <collision>
@@ -187,9 +176,5 @@
           filename="package://diff_robot_dan_description/meshes/shaft_left.STL" />
       </geometry>
-      <material
-        name="">
-        <color
-          rgba="0.64706 0.61961 0.58824 1" />
-      </material>
+      <material name="silver_metal"/>
     </visual>
     <collision>
@@ -243,9 +228,5 @@
           filename="package://diff_robot_dan_description/meshes/coupling_left.STL" />
       </geometry>
-      <material
-        name="">
-        <color
-          rgba="0.64706 0.51765 0 1" />
-      </material>
+      <material name="brass"/>
     </visual>
     <collision>
@@ -296,9 +277,5 @@
           filename="package://diff_robot_dan_description/meshes/ring_left.STL" />
       </geometry>
-      <material
-        name="">
-        <color
-          rgba="0 0 1 1" />
-      </material>
+      <material name="blue_metal"/>
     </visual>
     <collision>
@@ -349,9 +326,5 @@
           filename="package://diff_robot_dan_description/meshes/neumatic_left.STL" />
       </geometry>
-      <material
-        name="">
-        <color
-          rgba="0.29804 0.29804 0.29804 1" />
-      </material>
+      <material name="black"/>
     </visual>
     <collision>
@@ -402,9 +375,5 @@
           filename="package://diff_robot_dan_description/meshes/motor_support_right.STL" />
       </geometry>
-      <material
-        name="">
-        <color
-          rgba="0.89804 0.91765 0.92941 1" />
-      </material>
+      <material name="black"/>
     </visual>
     <collision>
@@ -455,9 +424,5 @@
           filename="package://diff_robot_dan_description/meshes/motor_right.STL" />
       </geometry>
-      <material
-        name="">
-        <color
-          rgba="0.89804 0.91765 0.92941 1" />
-      </material>
+      <material name="silver_metal"/>
     </visual>
     <collision>
@@ -508,9 +473,5 @@
           filename="package://diff_robot_dan_description/meshes/shaft_right.STL" />
       </geometry>
-      <material
-        name="">
-        <color
-          rgba="0.647058823529412 0.619607843137255 0.588235294117647 1" />
-      </material>
+      <material name="silver_metal"/>
     </visual>
     <collision>
@@ -564,9 +525,5 @@
           filename="package://diff_robot_dan_description/meshes/coupling_right.STL" />
       </geometry>
-      <material
-        name="">
-        <color
-          rgba="0.647058823529412 0.517647058823529 0 1" />
-      </material>
+      <material name="brass"/>
     </visual>
     <collision>
@@ -617,9 +574,5 @@
           filename="package://diff_robot_dan_description/meshes/ring_right.STL" />
       </geometry>
-      <material
-        name="">
-        <color
-          rgba="0 0 1 1" />
-      </material>
+      <material name="blue_metal"/>
     </visual>
     <collision>
@@ -670,9 +623,5 @@
           filename="package://diff_robot_dan_description/meshes/neumatic_right.STL" />
       </geometry>
-      <material
-        name="">
-        <color
-          rgba="0.298039215686275 0.298039215686275 0.298039215686275 1" />
-      </material>
+      <material name="black"/>
     </visual>
     <collision>
@@ -723,9 +672,5 @@
           filename="package://diff_robot_dan_description/meshes/battery_holder.STL" />
       </geometry>
-      <material
-        name="">
-        <color
-          rgba="0.25098 0.25098 0.25098 1" />
-      </material>
+      <material name="black"/>
     </visual>
     <collision>
@@ -776,9 +721,5 @@
           filename="package://diff_robot_dan_description/meshes/battery_1.STL" />
       </geometry>
-      <material
-        name="">
-        <color
-          rgba="0.161 0.435 1 1" />
-      </material>
+      <material name="blue_electronic"/>
     </visual>
     <collision>
@@ -829,9 +770,5 @@
           filename="package://diff_robot_dan_description/meshes/battery_2.STL" />
       </geometry>
-      <material
-        name="">
-        <color
-          rgba="0.161 0.435 1 1" />
-      </material>
+      <material name="blue_electronic"/>
     </visual>
     <collision>
@@ -882,9 +819,5 @@
           filename="package://diff_robot_dan_description/meshes/arduino.STL" />
       </geometry>
-      <material
-        name="">
-        <color
-          rgba="0.161 0.435 1 1" />
-      </material>
+      <material name="blue_electronic"/>
     </visual>
     <collision>
@@ -935,9 +868,5 @@
           filename="package://diff_robot_dan_description/meshes/driver.STL" />
       </geometry>
-      <material
-        name="">
-        <color
-          rgba="0.894 0.039 0 1" />
-      </material>
+      <material name="red_electronic"/>
     </visual>
     <collision>
@@ -988,9 +917,5 @@
           filename="package://diff_robot_dan_description/meshes/hex_support_s1.STL" />
       </geometry>
-      <material
-        name="">
-        <color
-          rgba="1 1 1 1" />
-      </material>
+      <material name="brass"/>
     </visual>
     <collision>
@@ -1041,9 +966,5 @@
           filename="package://diff_robot_dan_description/meshes/hex_support_s2.STL" />
       </geometry>
-      <material
-        name="">
-        <color
-          rgba="1 1 1 1" />
-      </material>
+      <material name="brass"/>
     </visual>
     <collision>
@@ -1094,9 +1015,5 @@
           filename="package://diff_robot_dan_description/meshes/hex_support_s3.STL" />
       </geometry>
-      <material
-        name="">
-        <color
-          rgba="1 1 1 1" />
-      </material>
+      <material name="brass"/>
     </visual>
     <collision>
@@ -1147,9 +1064,5 @@
           filename="package://diff_robot_dan_description/meshes/hex_support_s4.STL" />
       </geometry>
-      <material
-        name="">
-        <color
-          rgba="1 1 1 1" />
-      </material>
+      <material name="brass"/>
     </visual>
     <collision>
@@ -1200,9 +1113,5 @@
           filename="package://diff_robot_dan_description/meshes/center_wheel_support.STL" />
       </geometry>
-      <material
-        name="">
-        <color
-          rgba="0.64706 0.61961 0.58824 1" />
-      </material>
+      <material name="silver_metal"/>
     </visual>
     <collision>
@@ -1253,9 +1162,5 @@
           filename="package://diff_robot_dan_description/meshes/roll_support.STL" />
       </geometry>
-      <material
-        name="">
-        <color
-          rgba="0.64706 0.61961 0.58824 1" />
-      </material>
+      <material name="silver_metal"/>
     </visual>
     <collision>
@@ -1306,9 +1211,5 @@
           filename="package://diff_robot_dan_description/meshes/central_shaft.STL" />
       </geometry>
-      <material
-        name="">
-        <color
-          rgba="0.64706 0.61961 0.58824 1" />
-      </material>
+      <material name="silver_metal"/>
     </visual>
     <collision>
@@ -1359,9 +1260,5 @@
           filename="package://diff_robot_dan_description/meshes/central_wheel.STL" />
       </geometry>
-      <material
-        name="">
-        <color
-          rgba="0.25098 0.25098 0.25098 1" />
-      </material>
+      <material name="black"/>
     </visual>
     <collision>
@@ -1412,9 +1309,5 @@
           filename="package://diff_robot_dan_description/meshes/sup_platform.STL" />
       </geometry>
-      <material
-        name="">
-        <color
-          rgba="1 1 1 1" />
-      </material>
+      <material name="grey_pla"/>
     </visual>
     <collision>
@@ -1465,9 +1358,5 @@
           filename="package://diff_robot_dan_description/meshes/raspberry.STL" />
       </geometry>
-      <material
-        name="">
-        <color
-          rgba="0 0.741 0.098 1" />
-      </material>
+      <material name="green_electronic"/>
     </visual>
     <collision>
@@ -1518,9 +1407,5 @@
           filename="package://diff_robot_dan_description/meshes/lidar_base.STL" />
       </geometry>
-      <material
-        name="">
-        <color
-          rgba="0.752941176470588 0.752941176470588 0.752941176470588 1" />
-      </material>
+      <material name="grey_pla"/>
     </visual>
     <collision>
@@ -1571,9 +1456,5 @@
           filename="package://diff_robot_dan_description/meshes/lidar.STL" />
       </geometry>
-      <material
-        name="">
-        <color
-          rgba="0.250980392156863 0.250980392156863 0.250980392156863 1" />
-      </material>
+      <material name="black"/>
     </visual>
     <collision>
@@ -1624,9 +1505,5 @@
           filename="package://diff_robot_dan_description/meshes/power_bank_support.STL" />
       </geometry>
-      <material
-        name="">
-        <color
-          rgba="0.75294 0.75294 0.75294 1" />
-      </material>
+      <material name="grey_pla"/>
     </visual>
     <collision>
@@ -1677,9 +1554,5 @@
           filename="package://diff_robot_dan_description/meshes/power_bank.STL" />
       </geometry>
-      <material
-        name="">
-        <color
-          rgba="1 1 1 1" />
-      </material>
+      <material name="white"/>
     </visual>
     <collision>
@@ -1730,9 +1603,5 @@
           filename="package://diff_robot_dan_description/meshes/camera.STL" />
       </geometry>
-      <material
-        name="">
-        <color
-          rgba="0.25098 0.25098 0.25098 1" />
-      </material>
+      <material name="black"/>
     </visual>
     <collision>
@@ -1783,9 +1652,5 @@
           filename="package://diff_robot_dan_description/meshes/hex_support_m1.STL" />
       </geometry>
-      <material
-        name="">
-        <color
-          rgba="0.64706 0.51765 0 1" />
-      </material>
+      <material name="brass"/>
     </visual>
     <collision>
@@ -1836,9 +1701,5 @@
           filename="package://diff_robot_dan_description/meshes/hex_support_m2.STL" />
       </geometry>
-      <material
-        name="">
-        <color
-          rgba="0.647058823529412 0.517647058823529 0 1" />
-      </material>
+      <material name="brass"/>
     </visual>
     <collision>
@@ -1889,9 +1750,5 @@
           filename="package://diff_robot_dan_description/meshes/hex_support_m3.STL" />
       </geometry>
-      <material
-        name="">
-        <color
-          rgba="0.647058823529412 0.517647058823529 0 1" />
-      </material>
+      <material name="brass"/>
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
Commit message: Description: Adding Camera for description and simulation

File: diff_robot_dan_description/urdf/diff_robot_dan_core.urdf.xacro (robot description, xacro)
@@ -1582,5 +1582,5 @@
       <origin
         xyz="9.7623E-09 0.0001601 -0.0081003"
-        rpy="0 0 0" />
+        rpy="0 0 1.5707" />
       <mass
         value="0.02241" />
@@ -1596,5 +1596,5 @@
       <origin
         xyz="0 0 0"
-        rpy="0 0 0" />
+        rpy="0 0 1.5707" />
       <geometry>
         <mesh
@@ -1618,5 +1618,5 @@
     <origin
       xyz="0 0.15525 0.0323"
-      rpy="0 0 3.1416" />
+      rpy="0 0 1.5707" />
     <parent
       link="base_platform" />

File: diff_robot_dan_description/urdf/diff_robot_dan_sensors.xacro (robot description, xacro)
@@ -51,5 +51,40 @@
                 <output_type>sensor_msgs/LaserScan</output_type>
                 <frame_name>lidar_frame</frame_name>
-                <!--min_intensity>100.0</min_intensity-->
+            </plugin>
+        </sensor>
+    </gazebo>
+    <link name="camera_link"></link>
+    <joint name="camera_joint" type="fixed">
+        <parent link="camera"/>
+        <child link="camera_link"/>
+        <origin xyz="0.01 0 0" rpy="0 0 0"/>
+    </joint>
+    <link name="camera_link_optical"></link>
+    <joint name="camera_optical_joint" type="fixed">
+        <parent link="camera_link"/>
+        <child link="camera_link_optical"/>
+        <origin xyz="0 0 0" rpy="1.57 0 1.57"/>
+    </joint>
+    <gazebo reference="camera_link">
+        <material>Gazebo/FlatBlack</material>
+        <sensor name="camera_robot" type="camera">
+            <pose> 0 0 0 0 0 0 </pose>
+            <always_on>true</always_on>
+            <visualize>true</visualize>
+            <update_rate> 10 </update_rate>
+            <camera>
+                <horizontal_fov>1.089</horizontal_fov>
+                <image>
+                    <format>R8G8B8</format>
+                    <width>640</width>
+                    <height>480</height>
+                </image>
+                <clip>
+                    <near>0.05</near>
+                    <far>8.0</far>
+                </clip>
+            </camera>
+            <plugin name="camera_controller" filename="libgazebo_ros_camera.so">
+                <frame_name>camera_link_optical</frame_name>
             </plugin>
         </sensor>

Commit message: Description and Gazebo: Testing ros2 control searching for the cause of the bug with odometry and phantom move

File: diff_robot_dan_description/urdf/diff_robot_dan_core.urdf.xacro (robot description, xacro)
@@ -332,6 +332,5 @@
         rpy="0 0 0" />
       <geometry>
-        <mesh
-          filename="package://diff_robot_dan_description/meshes/neumatic_left.STL" />
+        <sphere radius="0.03394"/>
       </geometry>
     </collision>
@@ -629,6 +628,5 @@
         rpy="0 0 0" />
       <geometry>
-        <mesh
-          filename="package://diff_robot_dan_description/meshes/neumatic_right.STL" />
+        <sphere radius="0.03394"/>
       </geometry>
     </collision>

Commit message: BackUp: Making backup for Ubuntu reinstallation

File: diff_robot_dan_description/urdf/diff_robot_dan_core.urdf.xacro (robot description, xacro)
@@ -2,5 +2,5 @@
 <robot xmlns:xacro="http://www.ros.org/wiki/xacro">
   <xacro:include filename="$(find diff_robot_dan_description)/urdf/materials_and_colors.xacro"/>
-  <xacro:property name="caster_type" value="continuous" />
+  <xacro:property name="caster_type" value="fixed" />
   <link name="base_link"/>
   <link

Commit message: Description and Gazebo: Updated collision and controller spawners, pending test related with phantom move

File: diff_robot_dan_description/urdf/diff_robot_dan_core.urdf.xacro (robot description, xacro)
@@ -1264,6 +1264,5 @@
         rpy="0 0 0" />
       <geometry>
-        <mesh
-          filename="package://diff_robot_dan_description/meshes/central_wheel.STL" />
+        <sphere radius="0.0127"/>
       </geometry>
     </collision>

Commit message: Description: Correcting controller params and changing friction

File: diff_robot_dan_description/urdf/diff_robot_dan_core.urdf.xacro (robot description, xacro)
@@ -341,7 +341,7 @@
         rpy="1.5708 0 0" />
       <geometry>
-        <sphere radius="0.03394"/>
-        <!--mesh
-          filename="package://diff_robot_dan_description/meshes/neumatic_left.STL" /-->
+        <!--sphere radius="0.033475"/-->
+        <mesh
+          filename="package://diff_robot_dan_description/meshes/neumatic_left.STL" />
       </geometry>
     </collision>
@@ -639,7 +639,7 @@
         rpy="1.5708 0 0" />
       <geometry>
-        <sphere radius="0.03394"/>
-        <!--mesh
-          filename="package://diff_robot_dan_description/meshes/neumatic_right.STL" /-->
+        <!--sphere radius="0.033475"/-->
+        <mesh
+          filename="package://diff_robot_dan_description/meshes/neumatic_right.STL" />
       </geometry>
     </collision>

File: diff_robot_dan_description/urdf/diff_robot_dan_gazebo.xacro (robot description, xacro)
@@ -98,22 +98,14 @@
     </gazebo>
     <gazebo reference="central_wheel">
-        <mu1 value="0.01"/>
-        <mu2 value="0.01"/>
+        <mu1 value="0.005"/>
+        <mu2 value="0.005"/>
     </gazebo>
     <gazebo reference="neumatic_right">
-        <mu1 value="0.1"/>
-        <mu2 value="0.1"/>
-        <kp>1.0</kp>
-        <kd>0.0</kd>
-        <minDepth>0.001</minDepth>
-        <maxVel>0.2</maxVel>
+        <mu1 value="0.8"/>
+        <mu2 value="0.8"/>
     </gazebo>
     <gazebo reference="neumatic_left">
-        <mu1 value="0.1"/>
-        <mu2 value="0.1"/>
-        <kp>1.0</kp>
-        <kd>0.0</kd>
-        <minDepth>0.001</minDepth>
-        <maxVel>0.2</maxVel>
+        <mu1 value="0.8"/>
+        <mu2 value="0.8"/>
     </gazebo>
 </robot>

Commit message: Description: Chaning collision to check if contacts improve and the robot doesn't by strange contacts

File: diff_robot_dan_description/urdf/diff_robot_dan_core.urdf.xacro (robot description, xacro)
@@ -341,7 +341,7 @@
         rpy="1.5708 0 0" />
       <geometry>
-        <!--sphere radius="0.033475"/-->
-        <mesh
-          filename="package://diff_robot_dan_description/meshes/neumatic_left.STL" />
+        <sphere radius="0.033475"/>
+        <!--mesh
+          filename="package://diff_robot_dan_description/meshes/neumatic_left.STL" /-->
       </geometry>
     </collision>
@@ -639,7 +639,7 @@
         rpy="1.5708 0 0" />
       <geometry>
-        <!--sphere radius="0.033475"/-->
-        <mesh
-          filename="package://diff_robot_dan_description/meshes/neumatic_right.STL" />
+        <sphere radius="0.033475"/>
+        <!--mesh
+          filename="package://diff_robot_dan_description/meshes/neumatic_right.STL" /-->
       </geometry>
     </collision>

File: diff_robot_dan_description/urdf/diff_robot_dan_gazebo.xacro (robot description, xacro)
@@ -102,10 +102,10 @@
     </gazebo>
     <gazebo reference="neumatic_right">
-        <mu1 value="0.8"/>
-        <mu2 value="0.8"/>
+        <mu1 value="0.9"/>
+        <mu2 value="0.9"/>
     </gazebo>
     <gazebo reference="neumatic_left">
-        <mu1 value="0.8"/>
-        <mu2 value="0.8"/>
+        <mu1 value="0.9"/>
+        <mu2 value="0.9"/>
     </gazebo>
 </robot>

File: diff_robot_dan_description/urdf/diff_robot_dan_sensors.xacro (robot description, xacro)
@@ -13,5 +13,5 @@
             <pose> 0 0 0 0 0 0 </pose>
             <always_on>true</always_on>
-            <visualize>true</visualize>
+            <visualize>false</visualize>
             <update_rate> 30 </update_rate>
             <ray>

Commit message: Description: Adding voltage regultator and its support for model and gazebo

File: diff_robot_dan_description/urdf/diff_robot_dan_core.urdf.xacro (robot description, xacro)
@@ -505,5 +505,5 @@
       link="shaft_right" />
     <axis
-      xyz="0 0 1" />
+      xyz="0 0 -1" />
     <limit
       effort="1.0297"
@@ -1893,10 +1893,10 @@
         value="0" />
       <inertia
-        ixx="0"
-        ixy="0"
-        ixz="0"
-        iyy="0"
-        iyz="0"
-        izz="0" />
+        ixx="1.48922995829569E-06"
+        ixy="5.25911835519131E-15"
+        ixz="3.33245387880175E-12"
+        iyy="1.48922882572878E-06"
+        iyz="3.85848640885222E-13"
+        izz="5.17103684689375E-08" />
     </inertial>
     <visual>
@@ -1933,3 +1933,103 @@
       xyz="0 0 0" />
   </joint>
+  <link
+    name="voltage_regulator_support">
+    <inertial>
+      <origin
+        xyz="0 -0.01248 0.0062"
+        rpy="0 0 0" />
+      <mass
+        value="0.0063217" />
+      <inertia
+        ixx="1176.59E-9"
+        ixy="0.00000"
+        ixz="0.00000"
+        iyy="4434.68E-9"
+        iyz="5.48E-9"
+        izz="5594.9E-9" />
+    </inertial>
+    <visual>
+      <origin
+        xyz="0 0 0"
+        rpy="1.5707 0 0" />
+      <geometry>
+        <mesh
+          filename="package://diff_robot_dan_description/meshes/voltage_regulator_support_2.STL"
+          scale="0.001 0.001 0.001"/>
+      </geometry>
+      <material name="black"/>
+    </visual>
+    <collision>
+      <origin
+        xyz="0 0 0"
+        rpy="1.5707 0 0" />
+      <geometry>
+        <mesh
+          filename="package://diff_robot_dan_description/meshes/voltage_regulator_support_2.STL"
+          scale="0.001 0.001 0.001" />
+      </geometry>
+    </collision>
+  </link>
+  <joint
+    name="voltage_reg_support_to_base"
+    type="fixed">
+    <origin
+      xyz="-0.0485 -0.0815 0.0025"
+      rpy="0 0 0" />
+    <parent
+      link="base_platform" />
+    <child
+      link="voltage_regulator_support" />
+    <axis
+      xyz="0 0 0" />
+  </joint>
+  <link
+    name="voltage_regulator">
+    <inertial>
+      <origin
+        xyz="0.0012574 0.00088917 0.0063217"
+        rpy="0 0 0" />
+      <mass
+        value="0.0063217" />
+      <inertia
+        ixx="3.0667E-06"
+        ixy="-1.079E-07"
+        ixz="-7.1385E-08"
+        iyy="7.3036E-06"
+        iyz="-5.4148E-08"
+        izz="9.8754E-06" />
+    </inertial>
+    <visual>
+      <origin
+        xyz="0 0 0"
+        rpy="1.5707 0 0" />
+      <geometry>
+        <mesh
+          filename="package://diff_robot_dan_description/meshes/voltage_regulator.STL" />
+      </geometry>
+      <material name="blue_electronic"/>
+    </visual>
+    <collision>
+      <origin
+        xyz="0 0 0"
+        rpy="1.5707 0 0" />
+      <geometry>
+        <mesh
+          filename="package://diff_robot_dan_description/meshes/voltage_regulator.STL" />
+      </geometry>
+    </collision>
+  </link>
+  <joint
+    name="voltage_regulator_to_support"
+    type="fixed">
+    <origin
+      xyz="0.0485 -0.0075 0.0215"
+      rpy="0 0 0" />
+    <parent
+      link="voltage_regulator_support" />
+    <child
+      link="voltage_regulator" />
+    <axis
+      xyz="0 0 0" />
+  </joint>
 </robot>

File: diff_robot_dan_description/urdf/diff_robot_dan_gazebo.xacro (robot description, xacro)
@@ -97,4 +97,10 @@
         <material>Gazebo/DarkGrey</material>
     </gazebo>
+    <gazebo reference="voltage_regulator_support">
+        <material>Gazebo/Black</material>
+    </gazebo>
+    <gazebo reference="voltage_regulator">
+        <material>Gazebo/Blue</material>
+    </gazebo>
     <gazebo reference="central_wheel">
         <mu1 value="0.005"/>
